Commit message: Create simple-snake and springy-snake. Increase ground size.

File: envs/models/ground.urdf (robot description, URDF)
Before this commit: robot ground, 1 links, 0 joints
Links:
- link baseLink: geometry collision box size=100 100 0.1; visual box size=100 100 0.1

File: envs/models/simple-snakev0.urdf (robot description, URDF)
Before this commit: robot snake, 17 links, 16 joints
Links:
- removed link module_-1.0
- removed link module_0.0
- removed link module_1.0
- removed link module_10.0
- removed link module_11.0
- removed link module_12.0
- removed link module_13.0
- removed link module_14.0
- removed link module_15
- removed link module_2.0
- removed link module_3.0
- removed link module_4.0
- removed link module_5.0
- removed link module_6.0
- removed link module_7.0
- removed link module_8.0
- removed link module_9.0
- added link link_-1.0, mass 0.2; collision cylinder length=0.2 radius=0.025; visual cylinder length=0.2 radius=0.025
- added link link_0.0, mass 0.2; collision cylinder length=0.2 radius=0.025; visual cylinder length=0.2 radius=0.025
- added link link_1.0, mass 0.2; collision cylinder length=0.2 radius=0.025; visual cylinder length=0.2 radius=0.025
- added link link_2.0, mass 0.2; collision cylinder length=0.2 radius=0.025; visual cylinder length=0.2 radius=0.025
- added link link_3.0, mass 0.2; collision cylinder length=0.2 radius=0.025; visual cylinder length=0.2 radius=0.025
- added link link_4.0, mass 0.2; collision cylinder length=0.2 radius=0.025; visual cylinder length=0.2 radius=0.025
- added link link_5.0, mass 0.2; collision cylinder length=0.2 radius=0.025; visual cylinder length=0.2 radius=0.025
- added link link_6.0, mass 0.2; collision cylinder length=0.2 radius=0.025; visual cylinder length=0.2 radius=0.025
- added link link_7.0, mass 0.2; collision cylinder length=0.2 radius=0.025; visual cylinder length=0.2 radius=0.025
- added link link_8, mass 0.2; collision cylinder length=0.2 radius=0.025; visual cylinder length=0.2 radius=0.025
Joints:
- removed joint joint_10.0_9.0
- removed joint joint_11.0_10.0
- removed joint joint_12.0_11.0
- removed joint joint_13.0_12.0
- removed joint joint_14.0_13.0
- removed joint joint_15_14.0
- removed joint joint_8.0_7.0
- removed joint joint_9.0_8.0
- added joint joint_8_7.0: type revolute, parent link_8, child link_7.0, origin xyz=-0.2 0 0, axis 0 1 0, limit lower=-3.1415/2 upper=3.1415/2 effort=1000.0 velocity=10
- joint joint_0.0_-1.0: axis 1 0 0 -> 0 1 0; child module_-1.0 -> link_-1.0; limit lower=-1.57075 upper=1.57075 effort=1000.0 velocity=10 -> lower=-3.1415/2 upper=3.1415/2 effort=1000.0 velocity=10; origin xyz=0 0 -0.05 -> xyz=-0.2 0 0; parent module_0.0 -> link_0.0
- joint joint_1.0_0.0: axis 0 1 0 -> 1 0 0; child module_0.0 -> link_0.0; limit lower=-1.57075 upper=1.57075 effort=1000.0 velocity=10 -> lower=-3.1415/2 upper=3.1415/2 effort=1000.0 velocity=10; origin xyz=0 0 -0.05 -> xyz=-0.2 0 0; parent module_1.0 -> link_1.0
- joint joint_2.0_1.0: axis 1 0 0 -> 0 1 0; child module_1.0 -> link_1.0; limit lower=-1.57075 upper=1.57075 effort=1000.0 velocity=10 -> lower=-3.1415/2 upper=3.1415/2 effort=1000.0 velocity=10; origin xyz=0 0 -0.05 -> xyz=-0.2 0 0; parent module_2.0 -> link_2.0
- joint joint_3.0_2.0: axis 0 1 0 -> 1 0 0; child module_2.0 -> link_2.0; limit lower=-1.57075 upper=1.57075 effort=1000.0 velocity=10 -> lower=-3.1415/2 upper=3.1415/2 effort=1000.0 velocity=10; origin xyz=0 0 -0.05 -> xyz=-0.2 0 0; parent module_3.0 -> link_3.0
- joint joint_4.0_3.0: axis 1 0 0 -> 0 1 0; child module_3.0 -> link_3.0; limit lower=-1.57075 upper=1.57075 effort=1000.0 velocity=10 -> lower=-3.1415/2 upper=3.1415/2 effort=1000.0 velocity=10; origin xyz=0 0 -0.05 -> xyz=-0.2 0 0; parent module_4.0 -> link_4.0
- joint joint_5.0_4.0: axis 0 1 0 -> 1 0 0; child module_4.0 -> link_4.0; limit lower=-1.57075 upper=1.57075 effort=1000.0 velocity=10 -> lower=-3.1415/2 upper=3.1415/2 effort=1000.0 velocity=10; origin xyz=0 0 -0.05 -> xyz=-0.2 0 0; parent module_5.0 -> link_5.0
- joint joint_6.0_5.0: axis 1 0 0 -> 0 1 0; child module_5.0 -> link_5.0; limit lower=-1.57075 upper=1.57075 effort=1000.0 velocity=10 -> lower=-3.1415/2 upper=3.1415/2 effort=1000.0 velocity=10; origin xyz=0 0 -0.05 -> xyz=-0.2 0 0; parent module_6.0 -> link_6.0
- joint joint_7.0_6.0: axis 0 1 0 -> 1 0 0; child module_6.0 -> link_6.0; limit lower=-1.57075 upper=1.57075 effort=1000.0 velocity=10 -> lower=-3.1415/2 upper=3.1415/2 effort=1000.0 velocity=10; origin xyz=0 0 -0.05 -> xyz=-0.2 0 0; parent module_7.0 -> link_7.0

File: envs/models/snake.xacro (robot description, xacro)
@@ -2,16 +2,18 @@
 <robot name="snake" xmlns:xacro="http://www.ros.org/wiki/xacro">
 	<!-- snake properties -->
-	<xacro:property name="num_links" value ="5" />
-	<xacro:property name="link_length" value="0.5" />
+	<xacro:property name="num_links" value ="8" />
+	<xacro:property name="link_length" value="0.2" />
 	<xacro:property name="link_radius" value="0.025" />
 	<xacro:property name="link_mass" value="0.2" />
 	<xacro:property name="joint_friction" value="0.2" />
 	<xacro:property name="joint_damping" value="0.001" />
-	<xacro:property name="spring_mass" value="0.001" />
-	<xacro:property name="spring_inertia" value="0.0" />
+	<xacro:property name="spring_mass" value="0.01" />
+	<xacro:property name="spring_inertia" value="0.000006" />
 	<xacro:property name="pi" value="3.1415" />
 	<xacro:property name="joint_type" value="1" /> <!-- 1=simple_joint -1=springy_joint -->
+	<xacro:property name="joint_minLimit" value="-${pi}/2" />
+	<xacro:property name="joint_maxLimit" value="${pi}/2" />
 	<xacro:macro name="snake_link" params="number">
-		<link name="module_${number}">
+		<link name="link_${number}">
 			<collision>
 				<geometry>
@@ -27,6 +29,6 @@
 			</visual>
 			<inertial>
-				<origin xyz="-${link_length/2} 0 0" rpy="0 ${pi/2} 0" />
-				<mass value="0.159" />
+				<origin xyz="-${link_length/2} 0 0" rpy="0 0 0" />
+				<mass value="${link_mass}" />
 				<inertia ixx="0.00006" iyy="0.00006" izz="0.00006" ixy="0" ixz="0" iyz="0" />
 			</inertial>
@@ -45,8 +47,7 @@
 		<!-- Springy joint -->
 		<joint name="joint_${parent}_m" type="revolute">
-			<limit effort="1000.0" lower="0" upper="${pi}"
-				velocity="10" />
+			<limit effort="1000.0" lower="${joint_minLimit}" upper="${joint_maxLimit}" velocity="10" />
 			<dynamics damping="${joint_damping}" friction="${joint_friction}" />
-			<parent link="module_${parent}" />
+			<parent link="link_${parent}" />
 			<child link="spring_${parent}" />
 			<origin xyz="-${link_length} 0 0" />
@@ -56,5 +57,5 @@
 			<visual>
 				<geometry>
-					<cylinder length="${2*link_radius}" radius=".001" />
+					<cylinder length="${2*link_radius}" radius="0.001" />
 				</geometry>
 				<origin xyz="0 0 0" rpy="${pi} 0 0" />
@@ -62,14 +63,12 @@
 			<inertial>
 				<mass value="${spring_mass}" />
-				<inertia ixx="${spring_inertia}" ixy="0.0" ixz="0.0"
-					iyy="${spring_inertia}" iyz="0.0" izz="${spring_inertia}" />
+				<inertia ixx="${spring_inertia}" ixy="0.0" ixz="0.0" iyy="${spring_inertia}" iyz="0.0" izz="${spring_inertia}" />
 			</inertial>
 		</link>
 		<joint name="joint_${parent}_${child}" type="revolute">
-			<limit effort="1000.0" lower="0" upper="${pi}"
-				velocity="10" />
-			<!-- <dynamics damping="${damping}" friction="${friction}" /> -->
+			<limit effort="1000.0" lower="${joint_minLimit}" upper="${joint_maxLimit}" velocity="10" />
+			<dynamics damping="${joint_damping}" friction="${joint_friction}" />
 			<parent link="spring_${parent}" />
-			<child link="module_${child}" />
+			<child link="link_${child}" />
 			<origin xyz="0 0 0" rpy="0 0 0" />
 			<axis xyz="${axis}" />
@@ -80,9 +79,8 @@
 		<!-- Simple joint -->
 		<joint name="joint_${parent}_${child}" type="revolute">
-			<limit effort="1000.0" lower="0" upper="${pi}"
-				velocity="10" />
+			<limit effort="1000.0" lower="${joint_minLimit}" upper="${joint_maxLimit}" velocity="10" />
 			<dynamics damping="${joint_damping}" friction="${joint_friction}" />
-			<parent link="module_${parent}" />
-			<child link="module_${child}" />
+			<parent link="link_${parent}" />
+			<child link="link_${child}" />
 			<origin xyz="-${link_length} 0 0" />
 			<axis xyz="${axis}" />

File: envs/models/springy-snakev0.urdf (robot description, URDF)
Before this commit: robot snake, 33 links, 32 joints
Links:
- removed link module_-1.0
- removed link module_0.0
- removed link module_1.0
- removed link module_10.0
- removed link module_11.0
- removed link module_12.0
- removed link module_13.0
- removed link module_14.0
- removed link module_15
- removed link module_2.0
- removed link module_3.0
- removed link module_4.0
- removed link module_5.0
- removed link module_6.0
- removed link module_7.0
- removed link module_8.0
- removed link module_9.0
- removed link spring_10.0
- removed link spring_11.0
- removed link spring_12.0
- removed link spring_13.0
- removed link spring_14.0
- removed link spring_15
- removed link spring_8.0
- removed link spring_9.0
- added link link_-1.0, mass 0.2; collision cylinder length=0.2 radius=0.025; visual cylinder length=0.2 radius=0.025
- added link link_0.0, mass 0.2; collision cylinder length=0.2 radius=0.025; visual cylinder length=0.2 radius=0.025
- added link link_1.0, mass 0.2; collision cylinder length=0.2 radius=0.025; visual cylinder length=0.2 radius=0.025
- added link link_2.0, mass 0.2; collision cylinder length=0.2 radius=0.025; visual cylinder length=0.2 radius=0.025
- added link link_3.0, mass 0.2; collision cylinder length=0.2 radius=0.025; visual cylinder length=0.2 radius=0.025
- added link link_4.0, mass 0.2; collision cylinder length=0.2 radius=0.025; visual cylinder length=0.2 radius=0.025
- added link link_5.0, mass 0.2; collision cylinder length=0.2 radius=0.025; visual cylinder length=0.2 radius=0.025
- added link link_6.0, mass 0.2; collision cylinder length=0.2 radius=0.025; visual cylinder length=0.2 radius=0.025
- added link link_7.0, mass 0.2; collision cylinder length=0.2 radius=0.025; visual cylinder length=0.2 radius=0.025
- added link link_8, mass 0.2; collision cylinder length=0.2 radius=0.025; visual cylinder length=0.2 radius=0.025
- added link spring_8, mass 0.01; visual cylinder length=0.05 radius=0.001
- link spring_0.0: mass 0.001 -> 0.01; geometry visual cylinder length=0.05 radius=0.001
- link spring_1.0: mass 0.001 -> 0.01; geometry visual cylinder length=0.05 radius=0.001
- link spring_2.0: mass 0.001 -> 0.01; geometry visual cylinder length=0.05 radius=0.001
- link spring_3.0: mass 0.001 -> 0.01; geometry visual cylinder length=0.05 radius=0.001
- link spring_4.0: mass 0.001 -> 0.01; geometry visual cylinder length=0.05 radius=0.001
- link spring_5.0: mass 0.001 -> 0.01; geometry visual cylinder length=0.05 radius=0.001
- link spring_6.0: mass 0.001 -> 0.01; geometry visual cylinder length=0.05 radius=0.001
- link spring_7.0: mass 0.001 -> 0.01; geometry visual cylinder length=0.05 radius=0.001
Joints:
- removed joint joint_10.0_9.0
- removed joint joint_10.0_m
- removed joint joint_11.0_10.0
- removed joint joint_11.0_m
- removed joint joint_12.0_11.0
- removed joint joint_12.0_m
- removed joint joint_13.0_12.0
- removed joint joint_13.0_m
- removed joint joint_14.0_13.0
- removed joint joint_14.0_m
- removed joint joint_15_14.0
- removed joint joint_15_m
- removed joint joint_8.0_7.0
- removed joint joint_8.0_m
- removed joint joint_9.0_8.0
- removed joint joint_9.0_m
- added joint joint_8_7.0: type revolute, parent spring_8, child link_7.0, origin xyz=0 0 0 rpy=0 0 0, axis 0 1 0, limit lower=-3.1415/2 upper=3.1415/2 effort=1000.0 velocity=10
- added joint joint_8_m: type revolute, parent link_8, child spring_8, origin xyz=-0.2 0 0, axis 0 1 0, limit lower=-3.1415/2 upper=3.1415/2 effort=1000.0 velocity=10
- joint joint_0.0_-1.0: axis 1 0 0 -> 0 1 0; child module_-1.0 -> link_-1.0; limit lower=-1.57075 upper=1.57075 effort=1000.0 velocity=10 -> lower=-3.1415/2 upper=3.1415/2 effort=1000.0 velocity=10
- joint joint_0.0_m: axis 1 0 0 -> 0 1 0; limit lower=-1.57075 upper=1.57075 effort=1000.0 velocity=10 -> lower=-3.1415/2 upper=3.1415/2 effort=1000.0 velocity=10; origin xyz=0 0 -0.05 -> xyz=-0.2 0 0; parent module_0.0 -> link_0.0
- joint joint_1.0_0.0: axis 0 1 0 -> 1 0 0; child module_0.0 -> link_0.0; limit lower=-1.57075 upper=1.57075 effort=1000.0 velocity=10 -> lower=-3.1415/2 upper=3.1415/2 effort=1000.0 velocity=10
- joint joint_1.0_m: axis 0 1 0 -> 1 0 0; limit lower=-1.57075 upper=1.57075 effort=1000.0 velocity=10 -> lower=-3.1415/2 upper=3.1415/2 effort=1000.0 velocity=10; origin xyz=0 0 -0.05 -> xyz=-0.2 0 0; parent module_1.0 -> link_1.0
- joint joint_2.0_1.0: axis 1 0 0 -> 0 1 0; child module_1.0 -> link_1.0; limit lower=-1.57075 upper=1.57075 effort=1000.0 velocity=10 -> lower=-3.1415/2 upper=3.1415/2 effort=1000.0 velocity=10
- joint joint_2.0_m: axis 1 0 0 -> 0 1 0; limit lower=-1.57075 upper=1.57075 effort=1000.0 velocity=10 -> lower=-3.1415/2 upper=3.1415/2 effort=1000.0 velocity=10; origin xyz=0 0 -0.05 -> xyz=-0.2 0 0; parent module_2.0 -> link_2.0
- joint joint_3.0_2.0: axis 0 1 0 -> 1 0 0; child module_2.0 -> link_2.0; limit lower=-1.57075 upper=1.57075 effort=1000.0 velocity=10 -> lower=-3.1415/2 upper=3.1415/2 effort=1000.0 velocity=10
- joint joint_3.0_m: axis 0 1 0 -> 1 0 0; limit lower=-1.57075 upper=1.57075 effort=1000.0 velocity=10 -> lower=-3.1415/2 upper=3.1415/2 effort=1000.0 velocity=10; origin xyz=0 0 -0.05 -> xyz=-0.2 0 0; parent module_3.0 -> link_3.0
- joint joint_4.0_3.0: axis 1 0 0 -> 0 1 0; child module_3.0 -> link_3.0; limit lower=-1.57075 upper=1.57075 effort=1000.0 velocity=10 -> lower=-3.1415/2 upper=3.1415/2 effort=1000.0 velocity=10
- joint joint_4.0_m: axis 1 0 0 -> 0 1 0; limit lower=-1.57075 upper=1.57075 effort=1000.0 velocity=10 -> lower=-3.1415/2 upper=3.1415/2 effort=1000.0 velocity=10; origin xyz=0 0 -0.05 -> xyz=-0.2 0 0; parent module_4.0 -> link_4.0
- joint joint_5.0_4.0: axis 0 1 0 -> 1 0 0; child module_4.0 -> link_4.0; limit lower=-1.57075 upper=1.57075 effort=1000.0 velocity=10 -> lower=-3.1415/2 upper=3.1415/2 effort=1000.0 velocity=10
- joint joint_5.0_m: axis 0 1 0 -> 1 0 0; limit lower=-1.57075 upper=1.57075 effort=1000.0 velocity=10 -> lower=-3.1415/2 upper=3.1415/2 effort=1000.0 velocity=10; origin xyz=0 0 -0.05 -> xyz=-0.2 0 0; parent module_5.0 -> link_5.0
- joint joint_6.0_5.0: axis 1 0 0 -> 0 1 0; child module_5.0 -> link_5.0; limit lower=-1.57075 upper=1.57075 effort=1000.0 velocity=10 -> lower=-3.1415/2 upper=3.1415/2 effort=1000.0 velocity=10
- joint joint_6.0_m: axis 1 0 0 -> 0 1 0; limit lower=-1.57075 upper=1.57075 effort=1000.0 velocity=10 -> lower=-3.1415/2 upper=3.1415/2 effort=1000.0 velocity=10; origin xyz=0 0 -0.05 -> xyz=-0.2 0 0; parent module_6.0 -> link_6.0
- joint joint_7.0_6.0: axis 0 1 0 -> 1 0 0; child module_6.0 -> link_6.0; limit lower=-1.57075 upper=1.57075 effort=1000.0 velocity=10 -> lower=-3.1415/2 upper=3.1415/2 effort=1000.0 velocity=10
- joint joint_7.0_m: axis 0 1 0 -> 1 0 0; limit lower=-1.57075 upper=1.57075 effort=1000.0 velocity=10 -> lower=-3.1415/2 upper=3.1415/2 effort=1000.0 velocity=10; origin xyz=0 0 -0.05 -> xyz=-0.2 0 0; parent module_7.0 -> link_7.0
