Commit message: Update Snake urdfs.

File: envs/models/simple-snakev0.urdf (robot description, URDF)
Before this commit: robot snake, 10 links, 9 joints
Joints:
- joint joint_0.0_-1.0: limit lower=-3.1415/2 upper=3.1415/2 effort=1000.0 velocity=10 -> lower=-1.57075 upper=1.57075 effort=1000.0 velocity=10
- joint joint_1.0_0.0: limit lower=-3.1415/2 upper=3.1415/2 effort=1000.0 velocity=10 -> lower=-1.57075 upper=1.57075 effort=1000.0 velocity=10
- joint joint_2.0_1.0: limit lower=-3.1415/2 upper=3.1415/2 effort=1000.0 velocity=10 -> lower=-1.57075 upper=1.57075 effort=1000.0 velocity=10
- joint joint_3.0_2.0: limit lower=-3.1415/2 upper=3.1415/2 effort=1000.0 velocity=10 -> lower=-1.57075 upper=1.57075 effort=1000.0 velocity=10
- joint joint_4.0_3.0: limit lower=-3.1415/2 upper=3.1415/2 effort=1000.0 velocity=10 -> lower=-1.57075 upper=1.57075 effort=1000.0 velocity=10
- joint joint_5.0_4.0: limit lower=-3.1415/2 upper=3.1415/2 effort=1000.0 velocity=10 -> lower=-1.57075 upper=1.57075 effort=1000.0 velocity=10
- joint joint_6.0_5.0: limit lower=-3.1415/2 upper=3.1415/2 effort=1000.0 velocity=10 -> lower=-1.57075 upper=1.57075 effort=1000.0 velocity=10
- joint joint_7.0_6.0: limit lower=-3.1415/2 upper=3.1415/2 effort=1000.0 velocity=10 -> lower=-1.57075 upper=1.57075 effort=1000.0 velocity=10
- joint joint_8_7.0: limit lower=-3.1415/2 upper=3.1415/2 effort=1000.0 velocity=10 -> lower=-1.57075 upper=1.57075 effort=1000.0 velocity=10

File: envs/models/snake.xacro (robot description, xacro)
@@ -11,7 +11,7 @@
 	<xacro:property name="spring_inertia" value="0.000006" />
 	<xacro:property name="pi" value="3.1415" />
-	<xacro:property name="joint_type" value="1" /> <!-- 1=simple_joint -1=springy_joint -->
-	<xacro:property name="joint_minLimit" value="-${pi}/2" />
-	<xacro:property name="joint_maxLimit" value="${pi}/2" />
+	<xacro:property name="joint_type" value="-1" /> <!-- 1=simple_joint -1=springy_joint -->
+	<xacro:property name="joint_minLimit" value="-${pi/2}" />
+	<xacro:property name="joint_maxLimit" value="${pi/2}" />
 	<xacro:macro name="snake_link" params="number">
 		<link name="link_${number}">

File: envs/models/springy-snakev0.urdf (robot description, URDF)
Before this commit: robot snake, 19 links, 18 joints
Joints:
- joint joint_0.0_-1.0: limit lower=-3.1415/2 upper=3.1415/2 effort=1000.0 velocity=10 -> lower=-1.57075 upper=1.57075 effort=1000.0 velocity=10
- joint joint_0.0_m: limit lower=-3.1415/2 upper=3.1415/2 effort=1000.0 velocity=10 -> lower=-1.57075 upper=1.57075 effort=1000.0 velocity=10
- joint joint_1.0_0.0: limit lower=-3.1415/2 upper=3.1415/2 effort=1000.0 velocity=10 -> lower=-1.57075 upper=1.57075 effort=1000.0 velocity=10
- joint joint_1.0_m: limit lower=-3.1415/2 upper=3.1415/2 effort=1000.0 velocity=10 -> lower=-1.57075 upper=1.57075 effort=1000.0 velocity=10
- joint joint_2.0_1.0: limit lower=-3.1415/2 upper=3.1415/2 effort=1000.0 velocity=10 -> lower=-1.57075 upper=1.57075 effort=1000.0 velocity=10
- joint joint_2.0_m: limit lower=-3.1415/2 upper=3.1415/2 effort=1000.0 velocity=10 -> lower=-1.57075 upper=1.57075 effort=1000.0 velocity=10
- joint joint_3.0_2.0: limit lower=-3.1415/2 upper=3.1415/2 effort=1000.0 velocity=10 -> lower=-1.57075 upper=1.57075 effort=1000.0 velocity=10
- joint joint_3.0_m: limit lower=-3.1415/2 upper=3.1415/2 effort=1000.0 velocity=10 -> lower=-1.57075 upper=1.57075 effort=1000.0 velocity=10
- joint joint_4.0_3.0: limit lower=-3.1415/2 upper=3.1415/2 effort=1000.0 velocity=10 -> lower=-1.57075 upper=1.57075 effort=1000.0 velocity=10
- joint joint_4.0_m: limit lower=-3.1415/2 upper=3.1415/2 effort=1000.0 velocity=10 -> lower=-1.57075 upper=1.57075 effort=1000.0 velocity=10
- joint joint_5.0_4.0: limit lower=-3.1415/2 upper=3.1415/2 effort=1000.0 velocity=10 -> lower=-1.57075 upper=1.57075 effort=1000.0 velocity=10
- joint joint_5.0_m: limit lower=-3.1415/2 upper=3.1415/2 effort=1000.0 velocity=10 -> lower=-1.57075 upper=1.57075 effort=1000.0 velocity=10
- joint joint_6.0_5.0: limit lower=-3.1415/2 upper=3.1415/2 effort=1000.0 velocity=10 -> lower=-1.57075 upper=1.57075 effort=1000.0 velocity=10
- joint joint_6.0_m: limit lower=-3.1415/2 upper=3.1415/2 effort=1000.0 velocity=10 -> lower=-1.57075 upper=1.57075 effort=1000.0 velocity=10
- joint joint_7.0_6.0: limit lower=-3.1415/2 upper=3.1415/2 effort=1000.0 velocity=10 -> lower=-1.57075 upper=1.57075 effort=1000.0 velocity=10
- joint joint_7.0_m: limit lower=-3.1415/2 upper=3.1415/2 effort=1000.0 velocity=10 -> lower=-1.57075 upper=1.57075 effort=1000.0 velocity=10
- joint joint_8_7.0: limit lower=-3.1415/2 upper=3.1415/2 effort=1000.0 velocity=10 -> lower=-1.57075 upper=1.57075 effort=1000.0 velocity=10
- joint joint_8_m: limit lower=-3.1415/2 upper=3.1415/2 effort=1000.0 velocity=10 -> lower=-1.57075 upper=1.57075 effort=1000.0 velocity=10
