Commit message: Correct new phantomx morphology inertia tensors.

File: envs/models/phantomx/phantomx.urdf (robot description, URDF)
Before this commit: robot phantomx, 25 links, 24 joints
Links:
- link baseLink: geometry collision mesh filename=meshes/body_coll.STL scale=1 1 1; visual mesh filename=meshes/body_low.STL scale=1 1 1
- link c1_lf: geometry collision mesh filename=meshes/connect_coll.STL scale=1 1 1; visual mesh filename=meshes/connect_low.STL scale=1 1 1
- link c1_lm: geometry collision mesh filename=meshes/connect_coll.STL scale=1 1 1; visual mesh filename=meshes/connect_low.STL scale=1 1 1
- link c1_lr: geometry collision mesh filename=meshes/connect_coll.STL scale=1 1 1; visual mesh filename=meshes/connect_low.STL scale=1 1 1
- link c1_rf: geometry collision mesh filename=meshes/connect_coll.STL scale=1 1 1; visual mesh filename=meshes/connect_low.STL scale=1 1 1
- link c1_rm: geometry collision mesh filename=meshes/connect_coll.STL scale=1 1 1; visual mesh filename=meshes/connect_low.STL scale=1 1 1
- link c1_rr: geometry collision mesh filename=meshes/connect_coll.STL scale=1 1 1; visual mesh filename=meshes/connect_low.STL scale=1 1 1
- link c2_lf: geometry collision mesh filename=meshes/connect_coll.STL scale=1 1 1; visual mesh filename=meshes/connect_low.STL scale=1 1 1
- link c2_lm: geometry collision mesh filename=meshes/connect_coll.STL scale=1 1 1; visual mesh filename=meshes/connect_low.STL scale=1 1 1
- link c2_lr: geometry collision mesh filename=meshes/connect_coll.STL scale=1 1 1; visual mesh filename=meshes/connect_low.STL scale=1 1 1
- link c2_rf: geometry collision mesh filename=meshes/connect_coll.STL scale=1 1 1; visual mesh filename=meshes/connect_low.STL scale=1 1 1
- link c2_rm: geometry collision mesh filename=meshes/connect_coll.STL scale=1 1 1; visual mesh filename=meshes/connect_low.STL scale=1 1 1
- link c2_rr: geometry collision mesh filename=meshes/connect_coll.STL scale=1 1 1; visual mesh filename=meshes/connect_low.STL scale=1 1 1
- link thigh_lf: geometry collision mesh filename=meshes/thigh_l_coll.STL scale=1 1 1; visual mesh filename=meshes/thigh_l_low.STL scale=1 1 1
- link thigh_lm: geometry collision mesh filename=meshes/thigh_l_coll.STL scale=1 1 1; visual mesh filename=meshes/thigh_l_low.STL scale=1 1 1
- link thigh_lr: geometry collision mesh filename=meshes/thigh_l_coll.STL scale=1 1 1; visual mesh filename=meshes/thigh_l_low.STL scale=1 1 1
- link thigh_rf: geometry collision mesh filename=meshes/thigh_l_coll.STL scale=1 1 1; visual mesh filename=meshes/thigh_l_low.STL scale=1 1 1
- link thigh_rm: geometry collision mesh filename=meshes/thigh_l_coll.STL scale=1 1 1; visual mesh filename=meshes/thigh_l_low.STL scale=1 1 1
- link thigh_rr: geometry collision mesh filename=meshes/thigh_l_coll.STL scale=1 1 1; visual mesh filename=meshes/thigh_l_low.STL scale=1 1 1
- link tibia_lf: geometry collision mesh filename=meshes/tibia_l_coll.STL scale=1 1 1; visual mesh filename=meshes/tibia_l_low.STL scale=1 1 1
- link tibia_lm: geometry collision mesh filename=meshes/tibia_l_coll.STL scale=1 1 1; visual mesh filename=meshes/tibia_l_low.STL scale=1 1 1
- link tibia_lr: geometry collision mesh filename=meshes/tibia_l_coll.STL scale=1 1 1; visual mesh filename=meshes/tibia_l_low.STL scale=1 1 1
- link tibia_rf: geometry collision mesh filename=meshes/tibia_l_coll.STL scale=1 1 1; visual mesh filename=meshes/tibia_l_low.STL scale=1 1 1
- link tibia_rm: geometry collision mesh filename=meshes/tibia_l_coll.STL scale=1 1 1; visual mesh filename=meshes/tibia_l_low.STL scale=1 1 1
- link tibia_rr: geometry collision mesh filename=meshes/tibia_l_coll.STL scale=1 1 1; visual mesh filename=meshes/tibia_l_low.STL scale=1 1 1

File: envs/models/phantomx/phantomx.xacro (robot description, xacro)
@@ -38,6 +38,5 @@
 			<origin xyz="0 0 0" />
 			<mass value="0.97559947" />
-			<inertia ixx="3.1081800" ixy="-0.25460189" ixz="2.0318174"
-				iyy="6.3787776" iyz="0.16417863" izz="5.3316425" />
+			<inertia ixx="3.1081800" ixy="0" ixz="0" iyy="5.3787776" iyz="0" izz="3.3316425" />
 		</inertial>
 		<visual>
@@ -68,5 +67,5 @@
 				<origin xyz="0 -${connect_offset} 0" rpy="0 0 0" />
 				<mass value="0.024357719" />
-				<inertia ixx="0.0051411124" ixy="-0.00057530255" ixz="-0.000024729049" iyy="0.0081915737" iyz="-0.000019223094" izz="0.0041379812" />
+				<inertia ixx="0.0051411124" ixy="0" ixz="0" iyy="0.0081915737" iyz="0" izz="0.0041379812" />
 			</inertial>
 			<visual>
@@ -89,5 +88,5 @@
 				<origin xyz="0 -${connect_offset} 0" rpy="0 0 0" />
 				<mass value="0.024357719" />
-				<inertia ixx="0.0051411124" ixy="-0.00057530255" ixz="-0.000024729049" iyy="0.0081915737" iyz="-0.000019223094" izz="0.0041379812" />
+				<inertia ixx="0.0051411124" ixy="0" ixz="0" iyy="0.0081915737" iyz="0" izz="0.0041379812" />
 			</inertial>
 			<visual>
@@ -110,5 +109,5 @@
 				<origin xyz="0 0 0" rpy="0 0 0" />
 				<mass value="0.024357719" />
-				<inertia ixx="0.0051411124" ixy="-0.00057530255" ixz="-0.000024729049" iyy="0.0081915737" iyz="-0.000019223094" izz="0.0041379812" />
+				<inertia ixx="0.0051411124" ixy="0" ixz="0" iyy="0.0081915737" iyz="0" izz="0.0041379812" />
 			</inertial>
 			<visual>
@@ -131,5 +130,5 @@
 				<origin xyz="0 0 0" rpy="0 0 0" />
 				<mass value="0.024357719" />
-				<inertia ixx="0.0051411124" ixy="-0.00057530255" ixz="-0.000024729049" iyy="0.0081915737" iyz="-0.000019223094" izz="0.0041379812" />
+				<inertia ixx="0.0051411124" ixy="0" ixz="0" iyy="0.0081915737" iyz="0" izz="0.0041379812" />
 			</inertial>
 			<visual>
